File: sdvx pro micro.kicad_sch (KiCad schematic)
At the start: 0 parts

Commit message: complete refactor
Parts:
- added A1: RaspberryPi_Pico, Module:RaspberryPi_Pico_Common_Unspecified, symbol MCU_Module:RaspberryPi_Pico
- added C1: C_Small, Capacitor_THT:C_Disc_D4.3mm_W1.9mm_P5.00mm, symbol Device:C_Small
- added J1: BT A, Connector_JST:JST_XH_B4B-XH-A_1x04_P2.50mm_Vertical, symbol Connector_Generic:Conn_01x04
- added J10: ENC L, Connector_JST:JST_XH_B4B-XH-A_1x04_P2.50mm_Vertical, symbol Connector_Generic:Conn_01x04
- added J11: ENC R, Connector_JST:JST_XH_B4B-XH-A_1x04_P2.50mm_Vertical, symbol Connector_Generic:Conn_01x04
- added J2: BT B, Connector_JST:JST_XH_B4B-XH-A_1x04_P2.50mm_Vertical, symbol Connector_Generic:Conn_01x04
- added J3: BT C, Connector_JST:JST_XH_B4B-XH-A_1x04_P2.50mm_Vertical, symbol Connector_Generic:Conn_01x04
- added J4: BT D, Connector_JST:JST_XH_B4B-XH-A_1x04_P2.50mm_Vertical, symbol Connector_Generic:Conn_01x04
- added J5: FX L, Connector_JST:JST_XH_B4B-XH-A_1x04_P2.50mm_Vertical, symbol Connector_Generic:Conn_01x04
- added J6: FX R, Connector_JST:JST_XH_B4B-XH-A_1x04_P2.50mm_Vertical, symbol Connector_Generic:Conn_01x04
- added J7: Start, Connector_JST:JST_XH_B4B-XH-A_1x04_P2.50mm_Vertical, symbol Connector_Generic:Conn_01x04
- added J8: POT L, Connector_JST:JST_PH_B3B-PH-K_1x03_P2.00mm_Vertical, symbol Connector_Generic:Conn_01x03
- added J9: POT R, Connector_JST:JST_PH_B3B-PH-K_1x03_P2.00mm_Vertical, symbol Connector_Generic:Conn_01x03
- added Q1, Q2, Q3, Q4, Q5, Q6, Q7: BSS138, Package_TO_SOT_SMD:SOT-23, symbol Transistor_FET:BSS138
- added R1, R3: 1k, Resistor_THT:R_Axial_DIN0204_L3.6mm_D1.6mm_P7.62mm_Horizontal, symbol Device:R_Small_US
- added R2, R4: 2k, Resistor_THT:R_Axial_DIN0204_L3.6mm_D1.6mm_P7.62mm_Horizontal, symbol Device:R_Small_US
- added SW1: SW_SPDT_321, symbol Switch:SW_SPDT_321
Connections:
- new net: A1.22 (GPIO17), J10.3 (Pin_3), R3.2, R4.2
- new net: A1.16 (GPIO12), Q6.2 (S)
- new net: J9.2 (Pin_2), R3.1
- new net: A1.9 (GPIO6), J7.1 (Pin_1)
- new net: J8.2 (Pin_2), R1.1
- new net: A1.21 (GPIO16), J10.2 (Pin_2), R1.2, R2.2
- new net: A1.17 (GPIO13), Q7.2 (S)
- new net: A1.24 (GPIO18), J11.2 (Pin_2)
- new net: A1.25 (GPIO19), J11.3 (Pin_3)
- new net: A1.7 (GPIO5), J6.1 (Pin_1)
- new net: A1.10 (GPIO7), Q1.2 (S)
- new net: A1.11 (GPIO8), Q2.2 (S)
- new net: A1.1 (GPIO0), J1.1 (Pin_1)
- new net: A1.5 (GPIO3), J4.1 (Pin_1)
- new net: A1.6 (GPIO4), J5.1 (Pin_1)
- new net: A1.15 (GPIO11), Q5.2 (S)
- new net: A1.12 (GPIO9), Q3.2 (S)
- new net: A1.14 (GPIO10), Q4.2 (S)
- new net: A1.2 (GPIO1), J2.1 (Pin_1)
- new net: A1.4 (GPIO2), J3.1 (Pin_1)
- new net: A1.26 (GPIO20), SW1.1 (C)
- new net +5V: A1.40 (VBUS), C1.1, J10.1 (Pin_1), J11.1 (Pin_1), J8.1 (Pin_1), J9.1 (Pin_1), Q1.3 (D), Q2.3 (D), Q3.3 (D), Q4.3 (D), Q5.3 (D), Q6.3 (D), Q7.3 (D)
- new net AGND: J8.3 (Pin_3), J9.3 (Pin_3), R2.1, R4.1
- new net BT-A LED: J1.3 (Pin_3), Q1.1 (G)
- new net BT-B LED: J2.3 (Pin_3), Q2.1 (G)
- new net BT-C LED: J3.3 (Pin_3), Q3.1 (G)
- new net BT-D LED: J4.3 (Pin_3), Q4.1 (G)
- new net FX-L LED: J5.3 (Pin_3), Q5.1 (G)
- new net FX-R LED: J6.3 (Pin_3), Q6.1 (G)
- new net GND: A1.13 (GND), A1.18 (GND), A1.23 (GND), A1.28 (GND), A1.3 (GND), A1.38 (GND), A1.8 (GND), C1.2, J1.2 (Pin_2), J1.4 (Pin_4), J10.4 (Pin_4), J11.4 (Pin_4), J2.2 (Pin_2), J2.4 (Pin_4), J3.2 (Pin_2), J3.4 (Pin_4), J4.2 (Pin_2), J4.4 (Pin_4), J5.2 (Pin_2), J5.4 (Pin_4), J6.2 (Pin_2), J6.4 (Pin_4), J7.2 (Pin_2), J7.4 (Pin_4), SW1.2 (B)
- new net START LED: J7.3 (Pin_3), Q7.1 (G)
